Commit message: [Views] added some new views in views.py and added test cases for the following views. DetailedTable, Armchair, Sofa, Oven, Sides, Countertop, Cooktop, hotplate and Sink. Aloso took the Roots out of the logical-table.urdf

File: resources/urdf/logical-table.urdf (robot description, URDF)
Before this commit: robot logical-table, 6 links, 5 joints
Links:
- removed link table_root
Joints:
- removed joint left_front_leg_to_top
- removed joint left_front_to_back
- removed joint left_front_to_right_back
- removed joint left_front_to_right_front
- removed joint origin_to_left_front_leg
- added joint srface_to_right_front_leg: type fixed, parent surface, child right_front_leg, origin xyz=0.5 -0.5 -0.6
- added joint surfacd_to_left_back_leg: type fixed, parent surface, child left_back_leg, origin xyz=-0.5 0.5 -0.6
- added joint surface_to_left_front_leg: type fixed, parent surface, child left_front_leg, origin xyz=-0.5 -0.5 -0.625
- added joint surface_to_right_back_leg: type fixed, parent surface, child right_back_leg, origin xyz=0.5 0.5 -0.6

Commit message: [Views] PR adjustments

File: resources/urdf/logical-table.urdf (robot description, URDF)
Before this commit: robot logical-table, 5 links, 4 joints
Joints:
- removed joint srface_to_right_front_leg
- removed joint surfacd_to_left_back_leg
- added joint surface_to_left_back_leg: type fixed, parent surface, child left_back_leg, origin xyz=-0.5 0.5 -0.6
- added joint surface_to_right_front_leg: type fixed, parent surface, child right_front_leg, origin xyz=0.5 -0.5 -0.6
